Commit message: added istruction for visualization and functioning of lidar in gazebo and ros2(links, joints, bridge, etc)

File: src/bumperbot_description/urdf/bumperbot.urdf.xacro (robot description, xacro)
@@ -175,3 +175,28 @@
     <axis xyz="0 0 0" />
   </joint>
+  <link name="laser_link">
+   <inertial>
+      <origin xyz="-0.011945780406062 -0.000381929217680526 -0.0170649378129477" rpy="0 0 0" />
+      <mass value="0.073084435549317" />
+      <inertia ixx="1.96074931730795E-05" ixy="-3.62091076640009E-07" ixz="4.28230084046735E-07"
+      iyy="2.40983835136327E-05" iyz="1.50180909250652E-08" izz="4.14184164228595E-05" />
+    </inertial>
+    <visual>
+     <origin xyz="0 0 0" rpy="0 0 0" />
+      <geometry>
+        <mesh filename="package://bumperbot_description/meshes/laser_link.STL" />
+      </geometry>
+    </visual>
+    <collision>
+      <origin xyz="0 0 0" rpy="0 0 0" />
+      <geometry>
+        <mesh filename="package://bumperbot_description/meshes/laser_link.STL" />
+      </geometry>
+    </collision>
+  </link>
+  <joint name="laser_joint" type="fixed">
+    <origin xyz="0.0 0.0 0.1208" rpy="0 0 3.14"/>
+    <parent link="base_link" />
+    <child link="laser_link" />
+  </joint>
 </robot>

File: src/bumperbot_description/urdf/bumperbot_gazebo.xacro (robot description, xacro)
@@ -46,4 +46,8 @@
       <plugin filename="ignition-gazebo-imu-system" name="ignition::gazebo::systems::Imu">
       </plugin>
+      <!--Lidar plugin-->
+      <plugin filename="ignition-gazebo-sensors-system" name="ignition::gazebo::systems::Sensors">
+        <render_engine>ogre2</render_engine><!--we can set a parameter of the lidar plugin-->
+      </plugin>
     </xacro:if>
     <!-- ROS 2 Iron or above -->
@@ -53,4 +57,8 @@
       </plugin>
       <plugin filename="gz-sim-imu-system" name="gz::sim::systems::Imu">
+      </plugin>
+      <!--Lidar plugin-->
+      <plugin filename="gz-sim-sensors-system" name="gz::sim::systems::Sensors">
+        <render_engine>ogre2</render_engine>
       </plugin>
     </xacro:unless>
@@ -107,3 +115,33 @@
     </sensor>
   </gazebo>
+  <gazebo reference="laser_link">
+    <sensor name ="laser" type="gpu_lidar"><!--will use gpu to simulate rays-->
+      <!--let's set the param of the sensor for the plugin-->
+      <always_on>true</always_on>
+      <visualize>true</visualize>
+      <topic>scan</topic>
+      <update_rate>5</update_rate>
+      <gz_frame_id>laser_link</gz_frame_id>
+      <ray>
+        <scan>
+          <horizontal>
+            <samples>360</samples>
+            <resolution>1.0</resolution>
+            <min_angle>0.0</min_angle>
+            <max_angle>6.28</max_angle><!--360°-->
+          </horizontal>
+        </scan>
+        <range>
+          <min>0.12</min><!--meters-->
+          <max>12.0</max><!--meters-->
+          <resolution>0.02</resolution>
+        </range>
+        <noise><!--noise of the sensor-->
+          <type>gaussian</type>
+          <mean>0.0</mean>
+          <stddev>0.01</stddev>
+        </noise>
+      </ray>
+    </sensor>
+  </gazebo>
 </robot>

Commit message: laser max range limited in code, so we removed the problem of fake paviment. I added the rays as marker array to see the lidar rays completely

File: src/bumperbot_description/urdf/bumperbot.urdf.xacro (robot description, xacro)
@@ -23,4 +23,5 @@
         <mesh filename="package://bumperbot_description/meshes/base_link.STL" />
       </geometry>
+      <material name="black"/>
     </visual>
     <collision>
@@ -49,4 +50,5 @@
         <mesh filename="package://bumperbot_description/meshes/wheel_right_link.STL" />
       </geometry>
+      <material name="blue"/>
     </visual>
     <collision>
@@ -77,4 +79,5 @@
         <mesh filename="package://bumperbot_description/meshes/wheel_left_link.STL" />
       </geometry>
+      <material name="blue"/>
     </visual>
     <collision>
@@ -104,4 +107,5 @@
         <mesh filename="package://bumperbot_description/meshes/caster_front_link.STL" />
       </geometry>
+      <material name="silver"/>
     </visual>
     <collision>
@@ -131,4 +135,5 @@
         <mesh filename="package://bumperbot_description/meshes/caster_rear_link.STL" />
       </geometry>
+      <material name="silver"/>
     </visual>
     <collision>
@@ -158,7 +163,5 @@
         <mesh filename="package://bumperbot_description/meshes/imu_link.STL" />
       </geometry>
-      <material name="">
-        <color rgba="0.792156862745098 0.819607843137255 0.933333333333333 1" />
-      </material>
+      <material name="blue"/>
     </visual>
     <collision>
@@ -176,15 +179,17 @@
   </joint>
   <link name="laser_link">
-   <inertial>
+    <inertial>
       <origin xyz="-0.011945780406062 -0.000381929217680526 -0.0170649378129477" rpy="0 0 0" />
       <mass value="0.073084435549317" />
       <inertia ixx="1.96074931730795E-05" ixy="-3.62091076640009E-07" ixz="4.28230084046735E-07"
-      iyy="2.40983835136327E-05" iyz="1.50180909250652E-08" izz="4.14184164228595E-05" />
-    </inertial>
-    <visual>
-     <origin xyz="0 0 0" rpy="0 0 0" />
+               iyy="2.40983835136327E-05" iyz="1.50180909250652E-08"
+               izz="4.14184164228595E-05" />
+    </inertial>
+    <visual>
+      <origin xyz="0 0 0" rpy="0 0 0" />
       <geometry>
         <mesh filename="package://bumperbot_description/meshes/laser_link.STL" />
       </geometry>
+      <material name="dark_grey"/>
     </visual>
     <collision>
@@ -196,7 +201,20 @@
   </link>
   <joint name="laser_joint" type="fixed">
-    <origin xyz="0.0 0.0 0.1208" rpy="0 0 3.14"/>
+    <origin xyz="-0.0050526 -0.0023221 0.1208" rpy="0 0 3.14" />
     <parent link="base_link" />
     <child link="laser_link" />
-  </joint>
+    <axis xyz="0 0 0" />
+  </joint>
+  <material name="blue">
+    <color rgba="0 0 1 1"/>
+  </material>
+  <material name="black">
+    <color rgba="0 0 0 1"/>
+  </material>
+  <material name="silver">
+    <color rgba="0.79 0.82 0.93 1"/>
+  </material>
+  <material name="dark_grey">
+    <color rgba="0.3 0.3 0.3 1"/>
+  </material>
 </robot>

File: src/bumperbot_description/urdf/bumperbot_gazebo.xacro (robot description, xacro)
@@ -46,7 +46,6 @@
       <plugin filename="ignition-gazebo-imu-system" name="ignition::gazebo::systems::Imu">
       </plugin>
-      <!--Lidar plugin-->
       <plugin filename="ignition-gazebo-sensors-system" name="ignition::gazebo::systems::Sensors">
-        <render_engine>ogre2</render_engine><!--we can set a parameter of the lidar plugin-->
+        <render_engine>ogre2</render_engine>
       </plugin>
     </xacro:if>
@@ -58,5 +57,4 @@
       <plugin filename="gz-sim-imu-system" name="gz::sim::systems::Imu">
       </plugin>
-      <!--Lidar plugin-->
       <plugin filename="gz-sim-sensors-system" name="gz::sim::systems::Sensors">
         <render_engine>ogre2</render_engine>
@@ -115,7 +113,7 @@
     </sensor>
   </gazebo>
+  <!-- 2D Laser Sensor -->
   <gazebo reference="laser_link">
-    <sensor name ="laser" type="gpu_lidar"><!--will use gpu to simulate rays-->
-      <!--let's set the param of the sensor for the plugin-->
+    <sensor name="lidar" type="gpu_lidar">
       <always_on>true</always_on>
       <visualize>true</visualize>
@@ -123,24 +121,24 @@
       <update_rate>5</update_rate>
       <gz_frame_id>laser_link</gz_frame_id>
-      <ray>
+      <lidar>
         <scan>
           <horizontal>
             <samples>360</samples>
-            <resolution>1.0</resolution>
-            <min_angle>0.0</min_angle>
-            <max_angle>6.28</max_angle><!--360°-->
+            <resolution>1.00000</resolution>
+            <min_angle>0.000000</min_angle>
+            <max_angle>6.280000</max_angle>
           </horizontal>
         </scan>
         <range>
-          <min>0.12</min><!--meters-->
-          <max>12.0</max><!--meters-->
+          <min>0.120000</min>
+          <max>12.0</max>
           <resolution>0.02</resolution>
         </range>
-        <noise><!--noise of the sensor-->
+        <noise>
           <type>gaussian</type>
           <mean>0.0</mean>
           <stddev>0.01</stddev>
         </noise>
-      </ray>
+      </lidar>
     </sensor>
   </gazebo>
